Commit message: Add missing meshes and remove dependency on [realsense2_description].

File: urdf/_d435.urdf.xacro (robot description, xacro)
@@ -47,6 +47,5 @@
         <geometry>
           <!-- <box size="${d435_cam_width} ${d435_cam_height} ${d435_cam_depth}"/> -->
-          <mesh filename="package://realsense2_description/meshes/d435.dae" />
-          <!--<mesh filename="package://realsense2_description/meshes/d435/d435.dae" />-->
+          <mesh filename="package://fkie_realsense_description/meshes/d435.dae" />
         </geometry>
         <material name="aluminum"/>
